File: nanoNode_M.2.kicad_pcb (KiCad board)
At the start: 2 copper layers, 22 x 30 mm, 21 parts, among them J1 Bus_M.2_Socket_A, J2 Conn_01x02_Pin, J3 Conn_01x02_Pin, U1 CH32V203GxUx, U2 TMP102, U3 LSM6DSOX, U4 ATECC508A-MAHDA, Y1 Crystal_8MHz

Commit message: update and gitignore
Parts:
- added G***: LOGO, LOGO, F.Cu at (124.5, 54.0)
